File: LSDA/LSDA.kicad_sch (KiCad schematic)
At the start: 34 parts, among them Q1 BC547, Q2 BC547, U1 LM324

Commit message: Revision 2
Parts:
- removed C2: 10uF, diy-nabra:cel1, symbol Device:C_Polarized
- removed R12: 100k, diy-nabra:r3, symbol Device:R
- removed R13: 10k, diy-nabra:r3, symbol Device:R
- added C4, C5: 1uF, diy-nabra:cpoly105, symbol Device:C
- added R21, R24: 100k, diy-nabra:r3, symbol Device:R
- added R22, R23: 68k, diy-nabra:r3, symbol Device:R
- RV1: value B100K -> B25k
Connections:
- net +9V: now also R21.1, R23.1
- net GND: now also C4.2, C5.2, R22.2, R24.2; no longer R10.1
- net MIDO: now also R10.1
- net at U1.12 (+), U1.9 (-): now also R18.1, RV1.2, U1.1
- new net Vref1: C4.1, R21.2, R22.1, U1.10 (+)
- new net Vref2: C5.1, R23.2, R24.1, U1.13 (-)
Other:
- company: (none) -> Neil Massey
- title: (none) -> Dlopper LSDA
- moved on the sheet: D1, D2, Q1, Q2, R10, R11, R14, R15, R16, R17, R18, R19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
