File: LSDA_PCB/LSDA_PCB.kicad_pcb (KiCad board)
At the start: 2 copper layers, 81 parts, among them Q1 BC547, Q2 BC547, U1 LM324

Commit message: PCB version
Parts:
- removed the BT1 at (28.5, 144.8)
- removed the C1 at (36.7, 116.8)
- removed the C3 at (45.5, 133.6)
- removed the C4 at (50.5, 87.8)
- removed the C5 at (50.5, 113.4)
- removed the D1 at (56.4, 85.1)
- removed the D2 at (56.4, 116.8)
- removed the D3 at (22.7, 122.8)
- removed the Q1 at (44.7, 74.5)
- removed the Q2 at (41.8, 125.7)
- removed the R1 at (29.7, 111.1)
- removed the R10 at (29.1, 97.8)
- removed the R11 at (29.0, 80.7)
- removed the R14 at (40.5, 87.6)
- removed the R15 at (46.6, 77.8)
- removed the R16 at (43.7, 119.9)
- removed the R17 at (46.9, 125.1)
- removed the R18 at (36.7, 81.9)
- removed the R19 at (47.5, 82.9)
- removed the R2 at (29.0, 119.9)
- removed the R20 at (47.5, 118.4)
- removed the R21 at (47.5, 95.2)
- removed the R22 at (55.8, 97.8)
- removed the R23 at (48.1, 102.2)
- removed the R24 at (54.9, 107.4)
- removed the R3 at (39.3, 57.8)
- removed the R4 at (39.3, 71.6)
- removed the R5 at (26.6, 91.4)
- removed the R6 at (39.3, 144.1)
- removed the R7 at (85.0, 133.2)
- removed the R7 at (39.3, 130.2)
- removed the R7 at (34.2, 133.2)
- removed the R8 at (26.6, 95.9)
- removed the R9 at (25.3, 82.9)
- removed REF**: power-1n4001, diy-nabra:power-1n4001
- removed REF**: cel1, diy-nabra:cel1
- removed REF**: qnpn, diy-nabra:qnpn
- removed REF**: cpoly105, diy-nabra:cpoly105
- removed REF**: wnob, diy-nabra:wnob
- removed the RV1 at (29.9, 69.8)
- removed the TP1 at (55.1, 75.6)
- removed the TP2 at (36.7, 77.5)
- removed the TP3 at (55.1, 126.4)
- removed the U1 at (40.5, 108.0)
- moved BT1 61.5 mm to (43.7, 105.2), turned to 40 degrees
- moved C3 57.5 mm to (29.3, 97.2)
- moved C5 57.5 mm to (24.3, 77.0)
- moved R16 57.5 mm to (31.1, 83.5)
- moved R17 57.5 mm to (27.9, 88.7)
- moved R23 57.5 mm to (26.7, 65.8)
- moved R6 57.5 mm to (35.6, 107.7)
- moved R7 57.5 mm to (35.6, 93.8)
- moved C1 57.5 mm to (38.1, 80.4)
- moved C4 57.5 mm to (24.3, 51.4)
- moved Q1 57.5 mm to (30.1, 38.1), turned to 180 degrees
- moved Q2 57.5 mm to (33.0, 89.3)
- moved R1 57.5 mm to (45.1, 74.7)
- moved R10 57.5 mm to (45.7, 61.4)
- moved R15 57.5 mm to (28.2, 41.4)
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Routing:
- net GND: track 238.0 -> 0.00 mm
- net +9V: track 409.2 -> 204.3 mm
- net Net-(R6-Pad2): track 101.0 -> 49.9 mm
- net Net-(U1C--): track 91.1 -> 45.2 mm
- net Net-(R3-Pad2): track 73.0 -> 35.5 mm
- net Net-(U1A--): track 73.2 -> 36.4 mm
- net MIDO: track 47.7 -> 23.8 mm
- net Vref2: track 29.4 -> 14.7 mm
- net Vref1: track 29.1 -> 14.5 mm
- net Net-(R11-Pad1): track 27.1 -> 13.7 mm
- net Net-(R20-Pad2): track 23.0 -> 11.2 mm
- net Net-(R19-Pad2): track 21.2 -> 10.6 mm
- net Net-(U1B--): track 20.4 -> 10.2 mm
- net Net-(R16-Pad1): track 16.8 -> 8.38 mm
- net Net-(R14-Pad2): track 16.4 -> 8.19 mm
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- added copper zone on B.Cu, net GND
Other:
- board outline added: 41.9 x 99.1 mm
- board text removed: "10uF polarised cap"
- board text removed: "1n4001"
- board text removed: "1uF MLCC cap"
- board text removed: "B25k"
- board text removed: "BC547/8/9"
- board text removed: "This is the Dlopper, a control circuit. It outputs gates and control voltage due to light differentials."
